File: project_0/project0/_autosave-project0.kicad_pcb (KiCad board)
At the start: 2 copper layers, 7 parts

Commit message: añado el archivo que ignora las librerias y actualizo la info de la tesis, están todos los circuitos ya hechos, al menos en esquemático, revisar footprints
Parts:
- added U1: LM741, LM741_THT:LM741-THT, F.Cu at (149.7, 109.4)
Changed lines of the file:
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@@
+    )
+  )
+  (footprint "LM741_THT:LM741-THT" (layer "F.Cu")
+    (at 149.725 109.385)
+    (property "Sheetfile" "project0.kicad_sch")
+    (property "Sheetname" "")
+    (attr through_hole)
+    (fp_text reference "U1" (at 0 -0.5 unlocked) (layer "F.SilkS")
+      (effects (font (size 1 1) (thickness 0.15)))
+    )
+    (fp_text value "LM741" (at 0 1 unlocked) (layer "F.Fab")
+      (effects (font (size 1 1) (thickness 0.15)))
     )
   )
