File: smps_24v_15amp_ring/smps_artillery/smps_artillery.kicad_pcb (KiCad board)
At the start: 2 copper layers, 8 parts, among them U1 LM741

Commit message: proyecto_smps_artillery, ingeniería a la inversa.
Parts:
- removed U1: LM741, LM741_THT:LM741-THT
Changed lines of the file:
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@@
-    )
-  )
-  (footprint "LM741_THT:LM741-THT" (layer "F.Cu")
-    (at 149.725 109.385)
-    (property "Sheetfile" "project0.kicad_sch")
-    (property "Sheetname" "")
-    (attr through_hole)
-    (fp_text reference "U1" (at 0 -0.5 unlocked) (layer "F.SilkS")
-      (effects (font (size 1 1) (thickness 0.15)))
-    )
-    (fp_text value "LM741" (at 0 1 unlocked) (layer "F.Fab")
-      (effects (font (size 1 1) (thickness 0.15)))
     )
   )
