File: power_supply_pm17VDC/power_supply_17VDC_low_noise/power_supply_17VDC_low_noise.kicad_sch (KiCad schematic)
At the start: 36 parts, among them J1 Terminal_01x03, J2 Terminal_01x04, U1 LM317, U2 LM337, U3 LM7812, U4 LM7805

Commit message: finalizado STM y fuente de poder limpia, todo conforme a las huellas.
Parts:
- C1, C2: footprint Capacitor_THT:CP_Radial_D13.0mm_P5.00mm -> Capacitor_THT:CP_Radial_D18.0mm_P7.50mm
Changed lines of the file:
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@@
 			)
 		)
-		(property "Footprint" "Capacitor_THT:CP_Radial_D13.0mm_P5.00mm"
+		(property "Footprint" "Capacitor_THT:CP_Radial_D18.0mm_P7.50mm"
 			(at 67.0052 64.77 0)
 			(effects
@@
 			)
 		)
-		(property "Footprint" "Capacitor_THT:CP_Radial_D13.0mm_P5.00mm"
+		(property "Footprint" "Capacitor_THT:CP_Radial_D18.0mm_P7.50mm"
 			(at 67.0052 76.2 0)
 			(effects

Commit message: chore: aplicar .gitignore y limpiar los archivos temporales de kiCad
Parts:
- removed J2: Terminal_01x04, TerminalBlock:TerminalBlock_MaiXu_MX126-5.0-04P_1x04_P5.00mm, symbol Connector:Screw_Terminal_01x04
- added J2, J3: Screw_Terminal_01x02, TerminalBlock_Phoenix:TerminalBlock_Phoenix_MKDS-1,5-2_1x02_P5.00mm_Horizontal, symbol Connector:Screw_Terminal_01x02
- J1: footprint Connector_JST:JST_NV_B03P-NV_1x03_P5.00mm_Vertical -> TerminalBlock_Phoenix:TerminalBlock_Phoenix_MKDS-1,5-3_1x03_P5.00mm_Horizontal
Connections:
- net GND: now also J2.2 (Pin_2)
- net at C8.2, D2.1 (K), D3.2 (A)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: now also J2.1 (Pin_1)
- net at C7.1, D1.2 (A), D4.1 (K)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: now also J3.1 (Pin_1)
- net at D11.2: now also J1.3 (Pin_3); no longer J1.1 (Pin_1)
- net at D11.4: now also J1.1 (Pin_1); no longer J1.3 (Pin_3)
- net at C12.1, D10.2 (A), U4.3 (VO): now also J3.2 (Pin_2)
Other:
- moved on the sheet: C10, C11, C9, D10, D9, J1, U3, U4
