File: stm_v3/amplificador/bufferx2_suma_amplificador_/bufferx2_suma_amplificador_.kicad_pcb (KiCad board)
At the start: 2 copper layers, 199.8 x 154.2 mm, 134 parts, among them J1 ADS1115, J10 MCP4725_2C, J11 MCP4725_2F, J12 MCP4725_3C, J13 MCP4725_3F, J14 MCP4725_4C, J15 MCP4725_4F, J16 MCP4725_1F, J17 Screw_Terminal_01x04, J18 Sample, J19 signal_in, J2 MCP4725_VBIAS, J20 Terminal_01x02, J3 FC03, J4 muxL_1-12, J5 muxR_13-24, J6 espL_1-19, J7 espR_20-38, J8 Driver_motor, J9 MCP4725_1C, Q1 2N3904, Q2 2N3906, Q3 2N3904, Q4 2N3906, Q5 2N3904, Q6 2N3906, Q7 2N3904, Q8 2N3906, SW1 E stop, SW2 Retraction, U1 PC817, U10 TL074, U2 PC817, U4 TL074, U5 TL074, U6 TL074, U7 TL074, U8 TL071, U9 TL071

Commit message: finalizado STM y fuente de poder limpia, todo conforme a las huellas.
Parts:
- added C43: 100nF, Capacitor_THT:C_Rect_L9.0mm_W3.6mm_P7.50mm_MKT, F.Cu at (93.2, 68.5)
- C31, C32, C33, C34, C35, C36, C37, C38: footprint Capacitor_THT:C_Disc_D5.0mm_W2.5mm_P2.50mm -> Capacitor_THT:C_Disc_D3.0mm_W1.6mm_P2.50mm
- J17: value Screw_Terminal_01x04 -> Voltages_input
- J20: value Terminal_01x02 -> VCCMotor_01x02
- moved J2 5.90 mm to (110.8, 66.8)
- moved J3 5.56 mm to (81.2, 72.8)
Routing:
- net +3.3V: track 505.4 -> 523.3 mm
- net SCL_esp: track 140.3 -> 146.8 mm
- net SDA_esp: track 131.2 -> 137.1 mm
- net buffer_vbias: track 174.7 -> 168.8 mm
- net fc_03: track 35.8 -> 33.8 mm
- net 5VDC: track 109.2 -> 109.9 mm
