File: stm_v3/circuits_all/circuits_all.kicad_sch (KiCad schematic)
At the start: 13 parts, among them J1 ESP32_left_conn, J10 Conn_01x06_Socket, J11 Conn_01x06_Socket, J12 Conn_01x06_Socket, J2 ESP32_right_conn, J3 MUX_left_conn, J4 MUX_right_conn, J5 Conn_01x06_Socket, J6 Conn_01x06_Socket, J7 Conn_01x06_Socket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

Commit message: chore: aplicar .gitignore y limpiar los archivos temporales de kiCad
Parts:
- removed J1: ESP32_left_conn, symbol Connector:Conn_01x19_Socket
- removed J2: ESP32_right_conn, symbol Connector:Conn_01x19_Socket
Other:
- moved on the sheet: J5, U1A, U1B, U1C, U1D
